File: panel/lp-01-panel.kicad_pcb (KiCad board)
At the start: 2 copper layers, 40.3 x 128.5 mm, 15 parts

Commit message: Revision A.2
- A few small component tweaks
- Add OSHW logos
- Prepare for public release?
Parts:
- added REF**: OSHW-Logo_7.5x8mm_SilkScreen, Symbol:OSHW-Logo_7.5x8mm_SilkScreen, B.Cu at (133.9, 60.1)
Other:
- board text added: "LP-01 Front Panel Rev A.2 robhailman.com"
- board text removed: "LP-01 Front Panel Rev A"
