File: lp-01_ota_low_pass_filter.sch (KiCad schematic (older format))
At the start: 48 parts, among them J1 AudioJack2, J2 AudioJack2, J3 AudioJack2, J4 AudioJack2, J5 Conn_02x05_Odd_Even, Q1 2N3906, Q2 2N3906, U1 TL072, U2 LM13700, U3 TL074

Commit message: Rev A1 - revised component values
Increase CV1 input impedance, and adjust values for V/oct at CV2
Parts:
- R18: value 100K -> 220K; MFN RNF18FTD100K -> RNMF14FTC220K
- RV4: value B10K -> B100K; MFN RD901F-40-15F-B10K-00DL1 (center detent) -> RD901F-40-15F-B100K-00DL1
Other:
- note added: "Trim procedure:\n\nRV3: resonance gain\n Reduce to minimum\n Increase until self-oscillation is sustained across frequency range at max resonance\nRV2: V/oct trim\n Set resonance (RV5) to self-oscillate\n Set so self-oscillation tracks 1 V/oct at J2 with no input in J2 or J3\n\nNotes on component values:\n\nD1-D2: LEDs with Vf around 2V recommended\nR1: frequency control (RV1) range limit - lower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"
- note removed: "Trim procedure:\n\nRV3: resonance gain\n Reduce to minimum\n Increase until self-oscillation is sustained across frequency range at max resonance\nRV2: V/oct trim\n Set resonance (RV5) to self-oscillate\n Set so self-oscillation tracks 1 V/oct at J1 with RV4 at center and no input in J2 or J3\n\nNotes on component values:\n\nD1-D2: LEDs with Vf around 2V recommended\nR1: frequency control (RV1) r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"
- note removed: "center detent"
Changed lines of the file:
@@
 EESchema Schematic File Version 4
-LIBS:lp-01_ota_low_pass_filter-cache
 EELAYER 30 0
 EELAYER END
@@
 Title "LP-01 OTA Low-Pass Filter"
 Date "2019-09-10"
-Rev "A"
+Rev "A.1"
 Comp "RJH"
 Comment1 ""
@@
 P 2300 2850
 F 0 "R18" V 2093 2850 50  0000 C CNN
-F 1 "100K" V 2184 2850 50  0000 C CNN
+F 1 "220K" V 2184 2850 50  0000 C CNN
 F 2 "Resistor_THT:R_Axial_DIN0204_L3.6mm_D1.6mm_P5.08mm_Horizontal" V 2230 2850 50  0001 C CNN
 F 3 "~" H 2300 2850 50  0001 C CNN
-F 4 "RNF18FTD100K" H 2300 2850 50  0001 C CNN "MFN"
+F 4 "RNMF14FTC220K" H 2300 2850 50  0001 C CNN "MFN"
 F 5 "Stackpole" H 2300 2850 50  0001 C CNN "Manufacturer"
 	1    2300 2850
@@
 Text Label 4200 3650 0    50   ~ 0
 I_ABC
-Text Notes 1800 2350 2    50   ~ 0
-center detent
 Connection ~ 2600 2200
 Wire Wire Line
@@
 P 1900 2200
 F 0 "RV4" H 1831 2154 50  0000 R CNN
-F 1 "B10K" H 1831 2245 50  0000 R CNN
+F 1 "B100K" H 1831 2245 50  0000 R CNN
 F 2 "Potentiometer_THT:Potentiometer_Alpha_RD901F-40-00D_Single_Vertical" H 1900 2200 50  0001 C CNN
 F 3 "~" H 1900 2200 50  0001 C CNN
-F 4 "RD901F-40-15F-B10K-00DL1 (center detent)" H 1900 2200 50  0001 C CNN "MFN"
+F 4 "RD901F-40-15F-B100K-00DL1" H 1900 2200 50  0001 C CNN "MFN"
 F 5 "Alpha" H 1900 2200 50  0001 C CNN "Manufacturer"
 	1    1900 2200
@@
 	1500 1050 1400 1050
 Text Notes 550  7950 0    50   ~ 0
-Trim procedure:\n\nRV3: resonance gain\n  Reduce to minimum\n  Increase until self-oscillation is sustained across frequency range at max resonance\nRV2: V/oct trim\n  Set resonance (RV5) to self-oscillate\n  Set so self-oscillation tracks 1 V/oct at J1 with RV4 at center and no input in J2 or J3\n\nNotes on component values:\n\nD1-D2: LEDs with Vf around 2V recommended\nR1: frequency control (RV1) range limit - lower values for higher range\nR2: frequency control (RV2) sensitivity - lower values for greater sensitivity\nR14: output gain - higher values for higher gain.\n  Higher values will cause clipping at self-oscillation, but give more gain if that is not desired\nR17: input gain reduction - higher values give higher output volume, with lower resonance\nR18: sensitivty of CV2 (untrimmed CV in) - lower values for greater sensitivity.\n  1V/oct at approx 240K\n
+Trim procedure:\n\nRV3: resonance gain\n  Reduce to minimum\n  Increase until self-oscillation is sustained across frequency range at max resonance\nRV2: V/oct trim\n  Set resonance (RV5) to self-oscillate\n  Set so self-oscillation tracks 1 V/oct at J2 with no input in J2 or J3\n\nNotes on component values:\n\nD1-D2: LEDs with Vf around 2V recommended\nR1: frequency control (RV1) range limit - lower values for higher range\nR2: frequency control (RV2) sensitivity - lower values for greater sensitivity\nR14: output gain - higher values for higher gain.\n  Higher values will cause clipping at self-oscillation, but give more gain if that is not desired\nR17: input gain reduction - higher values give higher output volume, with lower resonance\nR18: sensitivty of CV2 (untrimmed CV in) - lower values for greater sensitivity.
 Text Notes 550  6350 0    75   ~ 15
 Implementation Notes

Commit message: Revision A.2
- A few small component tweaks
- Add OSHW logos
- Prepare for public release?
Parts:
- added LOGO1: Logo_Open_Hardware_Large, Symbol:OSHW-Logo_5.7x6mm_SilkScreen, symbol Graphic:Logo_Open_Hardware_Large
- C1, C2: symbol Device:CP -> lp-01_ota_low_pass_filter-rescue:CP-Device; Vendor (none) -> Digi-Key
- C10, C11, C12, C3, C4, C5, C6, C7, C8, C9, D1, D2, Q1, Q2, R10, R11, R12, R13, R14, R15, R16, R17, R18, R19, R2, R3, R4, R5, R6, R7, R8, R9, U1, U2, U3: Vendor (none) -> Digi-Key
- J1, J2, J3, J4: Vendor (none) -> Thonk
- J5: MFN (none) -> 67997-410HLF; Manufacturer (none) -> Amphenol ICC / FCI; Vendor (none) -> Digi-Key
- R1: value 4K7 -> 47K; MFN RNMF14FTC4K70 -> RNMF14FTC47K0; Vendor (none) -> Digi-Key
- RV1: value B10K -> B100K; symbol Device:R_POT -> lp-01_ota_low_pass_filter-rescue:R_POT-Device; MFN RD901F-40-15F-B10K-00DL1 -> RD901F-40-15F-B100K; Vendor (none) -> Thonk
- RV2, RV3: symbol Device:R_POT_TRIM -> lp-01_ota_low_pass_filter-rescue:R_POT_TRIM-Device; Vendor (none) -> Digi-Key
- RV4: symbol Device:R_POT -> lp-01_ota_low_pass_filter-rescue:R_POT-Device; MFN RD901F-40-15F-B100K-00DL1 -> RD901F-40-15F-B100K; Vendor (none) -> Thonk
- RV5: value A100K -> B100K; symbol Device:R_POT -> lp-01_ota_low_pass_filter-rescue:R_POT-Device; MFN RD901F-40-15F-A100K -> RD901F-40-15F-B100K; Vendor (none) -> Thonk

Commit message: Revert RV5 to log pot
This works much better!
Parts:
- RV5: value B100K -> A100K; MFN RD901F-40-15F-B100K -> RD901F-40-15F-A100K
Changed lines of the file:
@@
 P 5950 5650
 F 0 "RV5" H 5880 5604 50  0000 R CNN
-F 1 "B100K" H 5880 5695 50  0000 R CNN
+F 1 "A100K" H 5880 5695 50  0000 R CNN
 F 2 "Potentiometer_THT:Potentiometer_Alpha_RD901F-40-00D_Single_Vertical" H 5950 5650 50  0001 C CNN
 F 3 "~" H 5950 5650 50  0001 C CNN
-F 4 "RD901F-40-15F-B100K" H 5950 5650 50  0001 C CNN "MFN"
+F 4 "RD901F-40-15F-A100K" H 5950 5650 50  0001 C CNN "MFN"
 F 5 "Alpha" H 5950 5650 50  0001 C CNN "Manufacturer"
 F 6 "Thonk" H 5950 5650 50  0001 C CNN "Vendor"
